File: _autosave-Xiao_Headers.kicad_sch (KiCad schematic)
At the start: 28 parts, among them J1 Barrel_Jack, P1 USB_C_Plug_USB2.0, SW1 SW_Push, SW2 SW_Push, U1 SHT4x, U2 ESP32-C3-WROOM-02, U3 TSL25911FN, U5 LT1963AxST-3.3

Commit message: Revised decoupling capacitor
Parts:
- added R14: 10k, symbol Device:R
- C5, C7: value 100nF -> 10μF
Connections:
- net +3V3: now also C5.1, C7.2, R3.2, SW2.1, U2.2 (EN), R14.1; no longer SW2.2
- net at SW1.2: now also C5.2; no longer C5.1
- net at C7.1, R11.2, U2.8 (IO9): now also SW2.2; no longer C7.2, SW2.1
- net at U2.7 (IO8): now also R14.2
- no-connect marks 2 -> 10
Other:
- moved on the sheet: C5, C7, P1, R11, R12, R13, R8, R9, SW1, SW2
