File: ESP32Seeed.kicad_sch (KiCad schematic)
At the start: 0 parts

Commit message: Final Design
Pushing it so I can make it into single layer on my PC
Other:
- sheet Xiao_Headers renamed Main board
- added sheet LuxAndSHT (LuxAndSHT.kicad_sch)
- sheet Main board: file Xiao_Headers.kicad_sch -> mainboard.kicad_sch
Changed lines of the file:
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@@
 	(paper "A4")
 	(sheet
-		(at 128.27 59.69)
+		(at 162.56 74.93)
+		(size 44.45 55.88)
+		(exclude_from_sim no)
+		(in_bom yes)
+		(on_board yes)
+		(dnp no)
+		(fields_autoplaced yes)
+		(stroke
+			(width 0.1524)
+			(type solid)
+		)
+		(fill
+			(color 0 0 0 0)
+		)
+		(property "Sheetname" "LuxAndSHT"
+			(at 162.56 74.2184 0)
+			(show_name no)
+			(do_not_autoplace no)
+			(effects
+				(font
+					(size 1.27 1.27)
+				)
+				(justify left bottom)
+			)
+		)
+		(property "Sheetfile" "LuxAndSHT.kicad_sch"
+			(at 162.56 131.3946 0)
+			(show_name no)
+			(do_not_autoplace no)
+			(effects
+				(font
+					(size 1.27 1.27)
+				)
+				(justify left top)
+			)
+		)
+		(instances
+			(project "ESP32Seeed"
+				(path "/ade8ac70-014a-4392-bd34-ea2a47fe814a"
+					(page "3")
+				)
+			)
+		)
+	)
+	(sheet
+		(at 82.55 74.93)
 		(size 45.72 54.61)
 		(exclude_from_sim no)
@@
 			(color 0 0 0 0)
 		)
-		(property "Sheetname" "Xiao_Headers"
-			(at 128.27 58.9784 0)
+		(property "Sheetname" "Main board"
+			(at 82.55 74.2184 0)
 			(show_name no)
 			(do_not_autoplace no)
@@
 			)
 		)
-		(property "Sheetfile" "Xiao_Headers.kicad_sch"
-			(at 128.27 114.8846 0)
+		(property "Sheetfile" "mainboard.kicad_sch"
+			(at 82.55 130.1246 0)
 			(show_name no)
 			(do_not_autoplace no)
