File: offgridsolarpanel.kicad_pcb (KiCad board)
At the start: 2 copper layers, 48 x 27.1 mm, 27 parts, among them J1 USB_C_Receptacle_USB2.0_14P, J2 Conn_01x04, J3 Conn_01x04, SW1 SW_Push, SW2 SW_Push, U1 SHT4x, U2 ESP32-C3-WROOM-02, U3 TSL25911FN, U5 LT1963AxST-3.3

Commit message: Modified board for production
Parts:
- moved C11 43.4 mm to (132.7, 125.3)
- moved C8 43.4 mm to (129.7, 125.3)
- moved C9 43.4 mm to (129.7, 125.3)
- moved U3 43.4 mm to (135.8, 125.2)
- moved C12 43.4 mm to (132.7, 125.3)
- moved U1 43.4 mm to (135.7, 125.2)
- moved J2 43.4 mm to (125.4, 127.2)
Other:
- board size 48 x 27.1 mm -> 23.2 x 35.9 mm
- board text added: "V-SCORE"
